Commit message: extra usbl updates

File: src/alpha_std_auv/alpha_std_description/urdf/base.urdf.xacro (robot description, xacro)
@@ -47,5 +47,5 @@
     <link name="usbl"/>
     <joint name="usbl_joint" type="fixed">
-        <origin xyz="0.0 0.0 0.0" rpy="3.1415926 0.0 -1.5707963"/>
+        <origin xyz="0.65 0.0 0.05" rpy="3.1415926 0.0 -1.5707963"/>
         <parent link="base_link"/>
         <child link="usbl"/>

File: src/alpha_std_auv/alpha_std_stonefish/description/alpha_std_follower.scn.xacro (robot description, xacro)
@@ -140,5 +140,5 @@
                 <link name="Base"/>
                 <origin rpy="3.1415926 0.0 0.0" xyz="-0.65 0.0 -0.05"/>
-                <noise angle="0.01 0.01 0.05" angular_velocity="0.05" yaw_drift="0.001" linear_acceleration="0.1"/>
+                <noise angle="0.0 0.0 0.0" angular_velocity="0.0" yaw_drift="0.00" linear_acceleration="0.0"/>
                 <ros_publisher topic="/${robot_name}/imu/stonefish/data"/>
             </sensor>
@@ -149,20 +149,20 @@
                 <ros_publisher topic="/${robot_name}/gps/fix"/>
             </sensor>
-            <comm name="USBL" device_id="2" type="usbl">
-                <link name="Base"/>
-                <autoping rate="1.0"/>
-                <origin rpy="0.0 0.0 0.0" xyz="0.0 0.0 0.0"/>
+            <comm name="usbl" device_id="3" type="usbl">
                 <specs min_vertical_fov="0.0" max_vertical_fov="360.0" range="1000.0"/>
                 <connect device_id="1" occlusion_test="false"/>
+                <autoping rate="1.0"/>
+                <noise range="0.1" horizontal_angle="0.0" vertical_angle="0.0"/>
+                <resolution range="0.1" angle="0.1"/>
+                <origin xyz="0.0 0.0 0.0" rpy="0.0 0.0 0.0"/>
+                <link name="Base"/>
                 <ros_publisher topic="/${robot_name}/usbl"/>
             </comm>
-            <!--
-            <comm name="Modem" device_id="4" type="acoustic_modem">
+            <!-- <comm name="Modem" device_id="4" type="acoustic_modem">
+                <specs min_vertical_fov="0.0" max_vertical_fov="360.0" range="1000.0"/>
+                <connect device_id="3" occlusion_test="true"/>
+                <origin xyz="0.0 0.0 0.0" rpy="0.0 0.0 0.0"/>
                 <link name="Base"/>
-                <origin rpy="0.0 -1.571 0.0" xyz="0.0 0.0 0.0"/>
-                <specs min_vertical_fov="0.0" max_vertical_fov="360.0" range="1000.0"/>
-                <connect device_id="2" occlusion_test="false"/>
-            </comm>
-            -->
+            </comm> -->
             <world_transform rpy="${rpy}" xyz="${xyz}"/>
         </robot>

File: src/alpha_std_auv/alpha_std_stonefish/scenarios/ocean_swarm.scn.xacro (robot description, xacro)
@@ -11,5 +11,5 @@
     <xacro:include filename="$(find alpha_std_stonefish)/description/alpha_std_follower.scn.xacro"/>
     <xacro:alpha_std_leader robot_name="leader" xyz="0.0 0.0 0.0" rpy="0.0 0.0 0.0"/>
-    <xacro:alpha_std_follower robot_name="follower" xyz="-5.0 0.0 0.0" rpy="0.0 0.0 0.0"/>
+    <xacro:alpha_std_follower robot_name="follower" xyz="-5.0 0.0 5.0" rpy="0.0 0.0 0.0"/>
     <environment>
         <ned latitude="41" longitude="71"/>

Commit message: rotated urdf to allign with stonefish data

File: src/alpha_std_auv/alpha_std_description/urdf/base.urdf.xacro (robot description, xacro)
@@ -47,5 +47,5 @@
     <link name="usbl"/>
     <joint name="usbl_joint" type="fixed">
-        <origin xyz="0.65 0.0 0.05" rpy="3.1415926 0.0 -1.5707963"/>
+        <origin xyz="0.65 0.0 0.0" rpy="0.0 -1.571 3.1415926"/>
         <parent link="base_link"/>
         <child link="usbl"/>
