Commit message: cleanup and rename

File: src/multi_vehicle_path_planning/alpha_swarm_description/urdf/base.urdf.xacro (robot description, xacro)
@@ -1,9 +1,9 @@
 <?xml version="1.0"?>
-<robot name="alpha_std" xmlns:xacro="http://ros.org/wiki/xacro">
+<robot name="alpha_swarm" xmlns:xacro="http://ros.org/wiki/xacro">
     <link name="base_link">
         <visual>
             <origin xyz="0.0 -0.63 -0.57" rpy="0.0 0.0 1.5707963"/>
             <geometry>
-                <mesh filename="package://alpha_std_description/mesh/alpha_std.stl" scale="0.001 0.001 0.001"/>
+                <mesh filename="package://alpha_swarm_description/mesh/alpha_std.stl" scale="0.001 0.001 0.001"/>
             </geometry>
         </visual>
@@ -47,5 +47,5 @@
     <link name="usbl"/>
     <joint name="usbl_joint" type="fixed">
-        <origin xyz="0.65 0.0 0.0" rpy="0.0 -1.571 3.1415926"/>
+        <origin xyz="0.65 0.0 0.0" rpy="0.0 0.0 0.0"/>
         <parent link="base_link"/>
         <child link="usbl"/>

File: src/multi_vehicle_path_planning/alpha_swarm_stonefish/description/alpha_swarm.scn.xacro (robot description, xacro)
@@ -8,6 +8,6 @@
 -->
 <scenario xmlns:xacro="http://ros.org/wiki/xacro">
-    <xacro:include filename="$(find alpha_std_stonefish)/description/looks.scn.xacro"/>
-    <xacro:include filename="$(find alpha_std_stonefish)/description/materials.scn.xacro"/>
+    <xacro:include filename="$(find alpha_swarm_stonefish)/description/looks.scn.xacro"/>
+    <xacro:include filename="$(find alpha_swarm_stonefish)/description/materials.scn.xacro"/>
     <xacro:macro name="alpha_leader" params="xyz rpy robot_name">
         <robot name="${robot_name}" fixed="false" self_collisions="false">
@@ -140,5 +140,5 @@
                 <link name="Base"/>
                 <origin rpy="3.1415926 0.0 0.0" xyz="-0.65 0.0 -0.05"/>
-                <noise angle="0.01 0.01 0.05" angular_velocity="0.05" yaw_drift="0.001" linear_acceleration="0.1"/>
+                <noise angle="0.0 0.0 0.0" angular_velocity="0.0" yaw_drift="0.00" linear_acceleration="0.0"/>
                 <ros_publisher topic="/${robot_name}/imu/stonefish/data"/>
             </sensor>
@@ -149,11 +149,4 @@
                 <ros_publisher topic="/${robot_name}/gps/fix"/>
             </sensor>
-            <comm name="Modem" device_id="1" type="acoustic_modem">
-                <specs min_vertical_fov="0.0" max_vertical_fov="360.0" range="1000.0"/>
-                <connect device_id="3" occlusion_test="false"/>
-                <origin xyz="0.0 0.0 0.0" rpy="0.0 0.0 0.0"/>
-                <link name="Base"/>
-                <ros_publisher topic="/${robot_name}/modem"/>
-            </comm>
             <comm name="Modem" device_id="1" type="acoustic_modem">
                 <specs min_vertical_fov="0.0" max_vertical_fov="360.0" range="1000.0"/>
@@ -306,10 +299,10 @@
             </sensor>
             <comm name="usbl" device_id="3" type="usbl">
-                <specs min_vertical_fov="0.0" max_vertical_fov="180.0" range="1000.0"/>
+                <specs min_vertical_fov="0.0" max_vertical_fov="360.0" range="1000.0"/>
                 <connect device_id="1" occlusion_test="false"/>
                 <autoping rate="1.0"/>
-                <noise range="0.1" horizontal_angle="0.1" vertical_angle="0.1"/>
+                <!-- <noise range="0.1" horizontal_angle="0.1" vertical_angle="0.1"/> -->
                 <resolution range="0.1" angle="0.1"/>
-                <origin xyz="0.0 0.0 0.0" rpy="0.0 1.571 0.0"/>
+                <origin xyz="0.0 0.0 0.0" rpy="3.1415926 0.0 0.0"/>
                 <link name="Base"/>
                 <ros_publisher topic="/${robot_name}/usbl"/>

File: src/multi_vehicle_path_planning/alpha_swarm_stonefish/scenarios/ocean_swarm.scn.xacro (robot description, xacro)
@@ -8,9 +8,7 @@
 -->
 <scenario xmlns:xacro="http://ros.org/wiki/xacro">
-    <xacro:include filename="$(find alpha_std_stonefish)/description/alpha_std.scn.xacro"/>
-    <xacro:alpha_std robot_name="bill" xyz="0.0 0.0 0.0" rpy="0.0 0.0 0.0"/>
-    <xacro:alpha_std robot_name="lin" xyz="5.0 0.0 0.0" rpy="0.0 0.0 0.0"/>
-    <xacro:alpha_std robot_name="emir" xyz="5.0 5.0 0.0" rpy="0.0 0.0 0.0"/>
-    <xacro:alpha_std robot_name="mingxi" xyz="0.0 5.0 0.0" rpy="0.0 0.0 0.0"/>
+    <xacro:include filename="$(find alpha_swarm_stonefish)/description/alpha_swarm.scn.xacro"/>
+    <xacro:alpha_leader robot_name="leader" xyz="0.0 0.0 0.0" rpy="0.0 0.0 0.0"/>
+    <xacro:alpha_follower robot_name="follower" xyz="-20.0 0.0 0.0" rpy="0.0 0.0 0.0"/>
     <environment>
         <ned latitude="41" longitude="71"/>
